File: circuit/xmega-8e5-switch/xmega-128a4u-switch/xmega-128a4u-switch.brd (EAGLE design)
At the start: 100 x 80 mm, 28 parts, among them IC1 XMEGA16A4A

Commit message: circuit 01
Parts:
- added R6: 15k, eagle-ltspice:R0805
- added R7: 0R, eagle-ltspice:R1206
- added U$7: PDI, fab:2X03SMD
- U$3, U$4, U$5, U$6: value NETPORT -> NETPORT_IDC_FULLFLIP; device fab:2X03SMD -> fab:2X04SMD
- moved R5 45.0 mm to (28.9, 33.0), turned to 270 degrees
- moved D1 1.59 mm to (53.3, 15.2)
- moved R1 0.95 mm to (69.5, 40.0)
- moved R4 0.45 mm to (66.7, 34.9)
- moved R3 0.45 mm to (61.0, 38.1)
- moved R2 0.45 mm to (64.1, 43.8)
- turned U$3 to 225 degrees
- turned U$4 to 315 degrees
- turned U$5 to 45 degrees
- turned U$6 to 135 degrees
Connections:
- new net N$5: IC1.35, R6.1, U$7.5
- new net N$6: IC1.34, U$7.1
- net +3V3: now also R6.2, U$3.2, U$3.7, U$4.2, U$4.7, U$5.2, U$5.7, U$6.2, U$6.7, U$7.2; no longer U$3.4, U$4.4, U$5.4, U$6.4
- net GND: now also R7.1, R7.2, U$3.1, U$3.8, U$4.1, U$4.8, U$5.1, U$5.8, U$6.1, U$6.8, U$7.6; no longer U$3.3, U$4.3, U$5.3, U$6.3
- net NP1BI: now also IC1.14, U$3.3; no longer IC1.16, U$3.1
- net NP1BO: now also IC1.16; no longer IC1.14
- net NP1TI: now also U$3.5; no longer U$3.2
- net NP1TO: now also U$3.4; no longer U$3.5
- net NP2BI: now also IC1.40, U$4.3; no longer IC1.42, U$4.1
- net NP2BO: now also IC1.42; no longer IC1.40
- net NP2TI: now also U$4.5; no longer U$4.2
- net NP2TO: now also U$4.4; no longer U$4.5
- net NP3BI: now also IC1.4, U$5.3; no longer IC1.6, U$5.1
- net NP3BO: now also IC1.6; no longer IC1.4
- net NP3TI: now also U$5.5; no longer U$5.2
- net NP3TO: now also U$5.4; no longer U$5.5
- net NP4BI: now also IC1.10, U$6.3; no longer IC1.12, U$6.1
- net NP4BO: now also IC1.12; no longer IC1.10
- net NP4TI: now also U$6.5; no longer U$6.2
- net NP4TO: now also U$6.4; no longer U$6.5
Routing:
- net +3V3: track 336.8 -> 367.8 mm
- net N$5: track 0.00 -> 14.2 mm
- net N$6: track 0.00 -> 12.5 mm
- net NP4BO: track 30.0 -> 20.4 mm
- net NP4BI: track 21.3 -> 29.9 mm
- net NP2BO: track 26.9 -> 19.2 mm
- net NP2BI: track 18.7 -> 26.2 mm
- net NP3BO: track 25.7 -> 18.7 mm
- net NP1BO: track 52.9 -> 47.8 mm
- net NP3BI: track 19.7 -> 24.5 mm
- net NP1BI: track 49.5 -> 54.1 mm
- net N$7: track 16.7 -> 13.3 mm
- net NP1TI: track 54.8 -> 51.9 mm
- net NP2_STAT: track 14.0 -> 15.3 mm
- net NP3TO: track 19.3 -> 18.4 mm
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- added copper zone on layer 16, net N$8
