File: circuit/xmega-8e5-switch/xmega-128a4u-switch/xmega-128a4u-switch.sch (EAGLE design)
At the start: 28 parts, among them IC1 XMEGA16A4A

Commit message: circuit 01
Parts:
- added R6: 15k, eagle-ltspice:R
- added R7: 0R, eagle-ltspice:RR1206
- added U$7: PDI, fab:PDI
- U$3, U$4, U$5, U$6: value NETPORT -> NETPORT_IDC_FULLFLIP; device fab:NETPORT -> fab:NETPORT_IDC_FULLFLIP
Connections:
- new net N$5: IC1.!RESET!/PDI_CLK, R6.1, U$7.PDI_CLK
- new net N$6: IC1.PDI_DATA, U$7.PDI_DATA
- net +3V3: now also R6.2, U$3.VCC1, U$3.VCC2, U$4.VCC1, U$4.VCC2, U$5.VCC1, U$5.VCC2, U$6.VCC1, U$6.VCC2, U$7.VCC; no longer U$3.VCC, U$4.VCC, U$5.VCC, U$6.VCC
- net GND: now also R7.1, R7.2, U$3.GND1, U$3.GND2, U$4.GND1, U$4.GND2, U$5.GND1, U$5.GND2, U$6.GND1, U$6.GND2, U$7.GND; no longer U$3.GND, U$4.GND, U$5.GND, U$6.GND
- net NP1BI: now also IC1.PC4; no longer IC1.PC6
- net NP1BO: now also IC1.PC6; no longer IC1.PC4
- net NP2BI: now also IC1.PA0; no longer IC1.PA2
- net NP2BO: now also IC1.PA2; no longer IC1.PA0
- net NP3BI: now also IC1.PB0; no longer IC1.PB2
- net NP3BO: now also IC1.PB2; no longer IC1.PB0
- net NP4BI: now also IC1.PC0; no longer IC1.PC2
- net NP4BO: now also IC1.PC2; no longer IC1.PC0
Other:
- moved on the sheet: C10, C3, C7, C8, C9, D1, U$2
