File: circuit/xmega-128a4u-switch/xmega-128a4u-switch/xmega-128a4u-switch.sch (EAGLE design)
At the start: 30 parts, among them IC1 XMEGA16A4A

Commit message: update proposal, draft 01 report 01, circuit, figures
Parts:
- removed C3, C6: 1uF, eagle-ltspice:C
- removed D2, D3, D4: CDBM1100-G, fab:CDBM1100-G
- removed U$1: FTDI-SMD-HEADER, fab:FTDI-SMD-HEADER
- removed U$2: MICRO-USB_1/64, fab:MICRO-USB_1/64
- added R10, R11, R7, R9: 0R, eagle-ltspice:RR1206
- added R5, R6, R8: 15k, eagle-ltspice:R
- added S2: (no value), fab:6MM_SWITCH6MM_SWITCH
- added U$7: PDI, fab:PDI
- C1: value 1uF -> 0.1uF
- IC1: value XMEGA16A4A -> ATXMEGA_A4U; device atmel:XMEGA16A4A -> fab:ATXMEGA_A4U
- R1, R2, R3, R4: value (none) -> 2k2; device eagle-ltspice:R -> eagle-ltspice:RR1206
- U$3, U$4, U$5, U$6: value NETPORT -> NETPORT_IDC_FULLFLIP; device fab:NETPORT -> fab:NETPORT_IDC_FULLFLIP
Connections:
- removed net D+: IC1.PD7, U$2.D+
- removed net D-: IC1.PD6, U$2.D-
- removed net NP1BI: IC1.PC7, U$3.BI
- removed net NP1BO: IC1.PC5, U$3.BO
- removed net NP1TI: IC1.PC6, U$3.TI
- removed net NP1TO: IC1.PC4, U$3.TO
- removed net NP2BI: IC1.PA3, U$4.BI
- removed net NP2BO: IC1.PA1, U$4.BO
- removed net NP2TI: IC1.PA2, U$4.TI
- removed net NP2TO: IC1.PA0, U$4.TO
- removed net NP3BI: IC1.PB3, U$5.BI
- removed net NP3BO: IC1.PB1, U$5.BO
- removed net NP3TI: IC1.PB2, U$5.TI
- removed net NP3TO: IC1.PB0, U$5.TO
- removed net NP4BI: IC1.PC3, U$6.BI
- removed net NP4BO: IC1.PC1, U$6.BO
- removed net NP4TI: IC1.PC2, U$6.TI
- removed net NP4TO: IC1.PC0, U$6.TO
- removed net RX: IC1.PE0, U$1.TXD
- removed net TX: IC1.PE1, U$1.RXD
- new net N$5: IC1.!RESET!/PDI_CLK, R6.1, U$7.PDI_CLK
- new net N$6: IC1.PDI_DATA, U$7.PDI_DATA
- new net N$9: IC1.PD1/XCK0, R8.1, S2.S, S2.S1
- new net NP1_RX: IC1.PC2/RXD0, U$3.BI, U$3.TI
- new net NP1_TX: IC1.PC3/TXD0, U$3.BO, U$3.TO
- new net NP2_RX: IC1.PC6/RXD1/MISO, U$4.BI, U$4.TI
- new net NP2_TX: IC1.PC7/TXD1/SCK, U$4.BO, U$4.TO
- new net NP3_RX: IC1.PD2/RXD0, U$5.BI, U$5.TI
- new net NP3_TX: IC1.PD3/TXD0, U$5.BO, U$5.TO
- new net NP4_RX: IC1.PD6/RXD1/MISO, U$6.BI, U$6.TI
- new net NP4_TX: IC1.PD7/TXD1/SCK, U$6.BO, U$6.TO
- new net NP5_RX: IC1.PE2/RXD0
- new net NP5_TX: IC1.PE3/TXD0
- net +3V3: now also R10.1, R10.2, R11.1, R11.2, R5.2, R6.2, R7.1, R7.2, R8.2, R9.1, R9.2, U$3.VCC1, U$3.VCC2, U$4.VCC1, U$4.VCC2, U$5.VCC1, U$5.VCC2, U$6.VCC1, U$6.VCC2, U$7.VCC; no longer C3.2, C6.2, D2.KATHODE, D3.KATHODE, D4.KATHODE, U$1.VCC, U$2.VBUS, U$3.VCC, U$4.VCC, U$5.VCC, U$6.VCC
- net GND: now also C8.1, C9.1, S2.P, S2.P1, U$3.GND1, U$3.GND2, U$4.GND1, U$4.GND2, U$5.GND1, U$5.GND2, U$6.GND1, U$6.GND2, U$7.GND; no longer C3.1, C6.1, D2.ANODE, D3.ANODE, D4.ANODE, U$1.GND, U$2.GND, U$3.GND, U$4.GND, U$5.GND, U$6.GND
- net N$7: now also IC1.PD0, R5.1; no longer IC1.PA5
- net NP1_STAT: now also IC1.PC4/CS; no longer IC1.PD1
- net NP2_STAT: now also IC1.PC5/XCK1/MOSI; no longer IC1.PD4
- net NP3_STAT: now also IC1.PD4/CS; no longer IC1.PD3
- net NP4_STAT: now also IC1.PD5/XCK1/MOSI; no longer IC1.PD2
Other:
- note removed: "swap such that double-loop power rails"
- moved on the sheet: C10, C7, C8, C9, D1, S1
