File: circuit/atsams70n-switch/atsams70n-switch/atsams70n-switch.sch (EAGLE design)
At the start: 21 parts

Commit message: new hardware
Parts:
- removed JP1: (no value), pinhead:PINHD-2X20
- removed JP2, JP3, JP4, JP5: (no value), pinhead:PINHD-2X4
- removed S2, S3: (no value), fab:6MM_SWITCH6MM_SWITCH
- removed U$10, U$11, U$7, U$8, U$9: LEDRGBNEW, fab:LEDRGBNEW
- removed U$12: MICRO-USB_1/100, fab:MICRO-USB_1/100
- removed U$2, U$3, U$4, U$5: ISL3177E, fab:ISL3177E
- removed U$6: TC2050-MCP-NL, tag-connect-2050:TC2050-MCP-NL
- added C1: 22uF, eagle-ltspice:C
- added C10, C11, C12, C2, C3, C4, C5, C6, C7, C8, C9: 0.1uF, eagle-ltspice:CC0603
- added C13, C14: 22pF, eagle-ltspice:CC0603
- added C15, C19, C24, C25, C26, C27, C28, C29: 22uF 12v, eagle-ltspice:C
- added C16: 10pF, eagle-ltspice:C
- added C17, C18: 4.7uF, eagle-ltspice:C
- added C20, C21, C22, C23: 0.47uF, eagle-ltspice:C
- added D1, D2, D3, D4, D5: LEDRGBNEW, fab:LEDRGBNEW
- added J1, J2, J3, J4: (no value), fab:CONN_04X2SHROUDED
- added J5: CONN_20X2, SparkFun-Connectors:CONN_20X2
- added L1, L2: 10uH, eagle-ltspice:L
- added R1, R10, R7, R8, R9: 1k, eagle-ltspice:R
- added R11, R12, R13, R14, R15, R16, R17, R18, R2, R3: 2k2, eagle-ltspice:R
- added R20: 10K, eagle-ltspice:R
- added R4, R5: 2R2, eagle-ltspice:R
- added R6: 5k62, eagle-ltspice:R
- added TP1: TC2050-MCP-NL, tag-connect-2050:TC2050-MCP-NL
- added U1: REGULATOR_SOT223, fab:REGULATOR_SOT223
- added U3, U4, U5, U6: ISL3177E, fab:ISL3177E
- added X1: MICRO-USB_1/100, fab:MICRO-USB_1/100
- Q1: value (none) -> 20MHz
- renumbered U$1 to U2
Connections:
- new net +3V3: C1.1, C19.1, C2.2, C20.1, C21.1, C22.1, C23.1, C25.1, C26.1, C27.1, C28.1, C29.2, C3.2, C4.2, C5.2, C6.2, D1.A2, D2.A2, D3.A2, D4.A2, D5.A2, J1.2, J1.7, J2.2, J2.7, J3.2, J3.7, J4.2, J4.7, J5.39, J5.4, J5.6, R20.2, R4.1, R5.1, TP1.VTREF, U1.OUT1, U1.OUT2, U2.VDDIN, U2.VDDIO1, U2.VDDIO2, U2.VDDIO3, U2.VDDIO4, U2.VDDUTMII, U3.VCC, U4.VCC, U5.VCC, U6.VCC
- new net +5V: C15.2, C24.2, J5.2, U1.IN, X1.VBUS
- new net B1: R20.1, S1.S, S1.S1, U2.PA15/PWMC0_PWML3
- new net DM: U2.USB_DM, X1.D-
- new net DP: U2.USB_DP, X1.D+
- new net GND: C1.2, C10.1, C11.1, C12.1, C13.1, C14.2, C15.1, C16.2, C17.2, C18.1, C19.2, C2.1, C20.2, C21.2, C22.2, C23.2, C24.1, C25.2, C26.2, C27.2, C28.2, C29.1, C3.1, C4.1, C5.1, C6.1, C7.1, C8.1, C9.1, J1.1, J1.8, J2.1, J2.8, J3.1, J3.8, J4.1, J4.8, J5.1, J5.3, J5.5, R3.1, R6.1, S1.P, S1.P1, TP1.!TRST, TP1.GND, TP1.NC, U1.GND, U2.GND1, U2.GND2, U2.GND3, U2.GND4, U2.GND5, U2.GND6, U2.VREFN, U3.GND, U4.GND, U5.GND, U6.GND, X1.GND
- new net MK-AFE0-1: J5.16, U2.PA21/AFE0_AD1
- new net MK-AFE0-6: J5.25, U2.PA17/AFE0_AD6
- new net MK-AFE0-7: J5.26, U2.PA18/AFE0_AD7
- new net MK-AFE0-8: J5.27, U2.PA19/PWMC0_PWML0/AFE0_AD8
- new net MK-AFE0-9: J5.28, U2.PA20/PWMC0_PWML1/AFE0_AD9
- new net MK-DAC: U2.PD0/DAC1
- new net MK-F0: J5.33
- new net MK-F1: J5.37
- new net MK-F2: J5.38
- new net MK-F3: J5.40
- new net MK-F4: J5.30, U2.PA23
- new net MK-F5: J5.29, U2.PA16/PWMC0_PWML2
- new net MK-PWM0H0: J5.14, U2.PA11/PWMC0_PWMH0
- new net MK-PWM1H0: J5.18, U2.PD2/PWMC1_PWMH0
- new net MK-PWM1H1: J5.20, U2.PD4/PWMC1_PWMH1
- new net MK-PWM1H2: J5.22, U2.PD6/PWMC1_PWMH2
- new net MK-PWM1H3: J5.24, U2.PD8/PWMC1_PWMH3
- new net MK-PWM1L0: J5.17, U2.PD1/PWMC1_PWMLO
- new net MK-PWM1L1: J5.19, U2.PD3/PWMC1_PWML1
- new net MK-PWM1L2: J5.21, U2.PD5/PWMC1_PWML2
- new net MK-PWM1L3: J5.23, U2.PD7/PWMC1_PWML3
- new net MK-SPI-CS1: J5.15, U2.PA31/SPI0_NPCS1
- new net MK-SPI-CS2: J5.13, U2.PD12/SPI0_NPCS2
- new net MK-SPI-MISO: J5.11, U2.PD20/SPI0_MISO
- new net MK-SPI-MOSI: J5.12, U2.PD21/SPI0_MOSI
- new net MK-SPI-SPCK: J5.10, U2.PD22_SPI0_SPCK
- new net MK-TWD2: J5.9, U2.PD27/SPI0_NPCS3/TWD2
- new net MK-URX3-TWCK2: J5.7, U2.PD28/URXD3/TWCK2
- new net MK-USART-CTS: J5.32, U2.PB2/SPI0_NPCS0/CTS0
- new net MK-USART-RTS: J5.31, U2.PB3/RTS0
- new net MK-USART-RX: J5.35, U2.PB0/RXD0
- new net MK-USART-SCK: J5.34, U2.PB13/DAC0/SCK0
- new net MK-USART-TX: J5.36, U2.PB1/TXD0
- new net MK-UTX3: J5.8, U2.PD30/UTXD3
- new net N$1: D5.CRED, R17.2
- new net N$10: C18.2, L2.2, U2.VDDPLLUSB
- new net N$11: C17.1, L1.2, U2.VREFP
- new net N$12: D1.CRED, R2.2
- new net N$13: J3.3, U5.A
- new net N$14: J3.4, U5.B
- new net N$15: J3.5, U5.Z
- new net N$16: J3.6, U5.Y
- new net N$17: D4.CRED, R15.2
- new net N$18: D4.CBLUE, R9.2
- new net N$19: D4.CGREEN, R16.2
- new net N$2: D5.CBLUE, R10.2
- new net N$20: J2.3, U4.A
- new net N$21: J2.4, U4.B
- new net N$22: J2.5, U4.Z
- new net N$23: J2.6, U4.Y
- new net N$24: D3.CRED, R13.2
- new net N$25: J4.3, U6.A
- new net N$26: J4.4, U6.B
- new net N$27: J4.5, U6.Z
- new net N$28: J4.6, U6.Y
- new net N$29: D3.CBLUE, R8.2
- new net N$3: D5.CGREEN, R18.2
- new net N$30: D3.CGREEN, R14.2
- new net N$31: J1.3, U3.A
- new net N$32: J1.4, U3.B
- new net N$33: J1.5, U3.Z
- new net N$34: J1.6, U3.Y
- new net N$35: D2.CRED, R11.2
- new net N$36: D2.CBLUE, R7.2
- new net N$37: D2.CGREEN, R12.2
- new net N$38: D1.CBLUE, R1.2
- new net N$39: D1.CGREEN, R3.2
- new net N$4: C13.2, Q1.2, U2.PB9/XIN
- new net N$5: C14.1, Q1.1, U2.PB8/XOUT
- new net N$7: C16.1, R6.2, U2.VBG
- new net N$8: L2.1, R4.2
- new net N$9: L1.1, R5.2
- new net P1LB: R10.1, U2.PA13/PWMC0_PWMH2
- new net P1LG: R18.1, U2.PA8/XOUT32
- new net P1LR: R17.1, U2.PA22
- new net P1RX: U2.PD25/URXD2, U6.RO
- new net P1TX: U2.PD26/UTXD2, U6.DI
- new net P2LB: R9.1, U2.PA28
- new net P2LG: R16.1, U2.PD9
- new net P2LR: R15.1, U2.PA30
- new net P2RX: U2.PA9/URXD0, U5.RO
- new net P2TX: U2.PA10/UTXD0, U5.DI
- new net P3LB: R8.1, U2.PD15
- new net P3LG: R14.1, U2.PA0/I2SC0_MCK
- new net P3LR: R13.1, U2.PD10/PWMC0_PWML0
- new net P3RX: U2.PA5/URXD1, U4.RO
- new net P3TX: U2.PA4/UTXD1/TWCK0, U4.DI
- new net P4LB: R7.1, U2.PA27
- new net P4LG: R12.1, U2.PD14
- new net P4LR: R11.1, U2.PD13
- new net P4RX: U2.PD18/URXD4, U3.RO
- new net P4TX: U2.PD19/UTXD4, U3.DI
- new net RESET: TP1.RESET, U2.NRST
- new net STLB: R1.1, U2.PA1/I2SC0_CK
- new net STLR: R2.1, U2.PD11/PWMC0_PWMH0
- new net TCK: TP1.TCK, U2.PB7/SWCLK/TCK
- new net TDI: TP1.TDI, U2.PB4/TDI/TWD1
- new net TDO: TP1.TDO, U2.PB5/TDO/TWCK1
- new net TMS: TP1.TMS, U2.PB6/SWDIO/TMS
- new net VDDCORE: C10.2, C11.2, C12.2, C7.2, C8.2, C9.2, U2.VDDCORE1, U2.VDDCORE2, U2.VDDCORE3, U2.VDDCORE4, U2.VDDOUT, U2.VDDPLL, U2.VDDUTMIC
Other:
- moved on the sheet: Q1, S1

Commit message: remove cdc
Connections:
- net TCK renamed TCK/SWCLK
- net TMS renamed TMS/SWDIO
Changed lines of the file:
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@@
 <segment>
 <pinref part="U2" gate="G$1" pin="NRST"/>
-<wire x1="25.4" y1="27.94" x2="17.78" y2="27.94" width="0.1524" layer="91"/>
-<label x="17.78" y="27.94" size="1.778" layer="95"/>
+<wire x1="25.4" y1="27.94" x2="5.08" y2="27.94" width="0.1524" layer="91"/>
+<label x="5.08" y="27.94" size="1.778" layer="95"/>
 </segment>
 </net>
@@
 </segment>
 </net>
-<net name="TCK" class="0">
-<segment>
-<pinref part="U2" gate="G$1" pin="PB7/SWCLK/TCK"/>
-<wire x1="25.4" y1="12.7" x2="17.78" y2="12.7" width="0.1524" layer="91"/>
-<label x="17.78" y="12.7" size="1.778" layer="95"/>
-</segment>
-<segment>
-<wire x1="-62.23" y1="3.81" x2="-54.61" y2="3.81" width="0.1524" layer="91"/>
-<label x="-59.69" y="3.81" size="1.778" layer="95"/>
-<pinref part="TP1" gate="G$1" pin="TCK"/>
-</segment>
-</net>
-<net name="TMS" class="0">
-<segment>
-<pinref part="U2" gate="G$1" pin="PB6/SWDIO/TMS"/>
-<wire x1="25.4" y1="10.16" x2="17.78" y2="10.16" width="0.1524" layer="91"/>
-<label x="17.78" y="10.16" size="1.778" layer="95"/>
-</segment>
-<segment>
-<wire x1="-62.23" y1="-1.27" x2="-54.61" y2="-1.27" width="0.1524" layer="91"/>
-<label x="-59.69" y="-1.27" size="1.778" layer="95"/>
-<pinref part="TP1" gate="G$1" pin="TMS"/>
-</segment>
-</net>
 <net name="TDO" class="0">
 <segment>
 <pinref part="U2" gate="G$1" pin="PB5/TDO/TWCK1"/>
-<wire x1="25.4" y1="7.62" x2="17.78" y2="7.62" width="0.1524" layer="91"/>
-<label x="17.78" y="7.62" size="1.778" layer="95"/>
+<wire x1="25.4" y1="7.62" x2="5.08" y2="7.62" width="0.1524" layer="91"/>
+<label x="5.08" y="7.62" size="1.778" layer="95"/>
 </segment>
 <segment>
@@
 <segment>
 <pinref part="U2" gate="G$1" pin="PB4/TDI/TWD1"/>
-<wire x1="25.4" y1="5.08" x2="17.78" y2="5.08" width="0.1524" layer="91"/>
-<label x="17.78" y="5.08" size="1.778" layer="95"/>
+<wire x1="25.4" y1="5.08" x2="5.08" y2="5.08" width="0.1524" layer="91"/>
+<label x="5.08" y="5.08" size="1.778" layer="95"/>
 </segment>
 <segment>
@@
 </segment>
 </net>
+<net name="TCK/SWCLK" class="0">
+<segment>
+<pinref part="U2" gate="G$1" pin="PB7/SWCLK/TCK"/>
+<wire x1="25.4" y1="12.7" x2="5.08" y2="12.7" width="0.1524" layer="91"/>
+<label x="5.08" y="12.7" size="1.778" layer="95"/>
+</segment>
+<segment>
+<wire x1="-62.23" y1="3.81" x2="-54.61" y2="3.81" width="0.1524" layer="91"/>
+<label x="-59.69" y="3.81" size="1.778" layer="95"/>
+<pinref part="TP1" gate="G$1" pin="TCK"/>
+</segment>
+</net>
+<net name="TMS/SWDIO" class="0">
+<segment>
+<pinref part="U2" gate="G$1" pin="PB6/SWDIO/TMS"/>
+<wire x1="25.4" y1="10.16" x2="5.08" y2="10.16" width="0.1524" layer="91"/>
+<label x="5.08" y="10.16" size="1.778" layer="95"/>
+</segment>
+<segment>
+<wire x1="-62.23" y1="-1.27" x2="-54.61" y2="-1.27" width="0.1524" layer="91"/>
+<label x="-59.69" y="-1.27" size="1.778" layer="95"/>
+<pinref part="TP1" gate="G$1" pin="TMS"/>
+</segment>
+</net>
